Commit message: Fixes materials and stuff
Signed-off-by: Franco Cipollone <franco.c@ekumenlabs.com>

File: andino_description/urdf/include/common_macros.urdf.xacro (robot description, xacro)
@@ -1,4 +1,32 @@
 <?xml version="1.0"?>
 <robot xmlns:xacro="http://www.ros.org/wiki/xacro">
+<!-- ===================== Material ============================================
+  RVIZ material RGBA definition.
+-->
+  <material name="yellow">
+    <color rgba="1 0.95 0 1"/>
+  </material>
+  <material name="blue">
+    <color rgba="0 0 1 1"/>
+  </material>
+  <material name="light_blue">
+    <color rgba="0 0.5 0.8 1"/>
+  </material>
+  <material name="black">
+    <color rgba="0 0 0 1"/>
+  </material>
+  <material name="white">
+    <color rgba="1 1 1 1"/>
+  </material>
+  <material name="red">
+    <color rgba="0.8 0.0 0.0 1.0"/>
+  </material>
+  <material name="silver">
+    <color rgba="0.79 0.82 0.93 1"/>
+  </material>
+  <material name="dark_grey">
+    <color rgba="0.02 0.02 0.02 1"/>
+  </material>
+<!-- ========================================================================-->
 <!-- ===================== Wheel xacro =========================================
   params:
@@ -38,5 +66,5 @@
          <cylinder radius="${wheel_props['radius']}" length="${wheel_props['length']}"/>
         </geometry>
-        <material name="red"/>
+        <material name="dark_grey"/>
       </visual>
     </xacro:if>
@@ -242,31 +270,3 @@
   </xacro:macro>
 <!-- ========================================================================-->
-<!-- ===================== Material ============================================
-  RVIZ material RGBA definition.
--->
-  <material name="yellow">
-    <color rgba="1 0.95 0 1"/>
-  </material>
-  <material name="blue">
-    <color rgba="0 0 1 1"/>
-  </material>
-  <material name="light_blue">
-    <color rgba="0 0.5 0.8 1"/>
-  </material>
-  <material name="black">
-    <color rgba="0 0 0 1"/>
-  </material>
-  <material name="white">
-    <color rgba="1 1 1 1"/>
-  </material>
-  <material name="red">
-    <color rgba="0.8 0.0 0.0 1.0"/>
-  </material>
-  <material name="silver">
-    <color rgba="0.79 0.82 0.93 1"/>
-  </material>
-  <material name="dark_grey">
-    <color rgba="0.3 0.3 0.3 1"/>
-  </material>
-<!-- ========================================================================-->
 </robot>

File: andino_description/urdf/include/common_sensors.urdf.xacro (robot description, xacro)
@@ -20,5 +20,5 @@
         <cylinder radius="${sensor_prop['laser']['radius']}" length="${sensor_prop['laser']['length']}"/>
       </geometry>
-      <material name="red"/>
+      <material name="dark_grey"/>
     </visual>
   </xacro:if>

File: andino_gz/urdf/andino_gz.urdf.xacro (robot description, xacro)
@@ -14,3 +14,4 @@
     </plugin>
   </gazebo>
+  <!-- <xacro:include filename="$(find andino_gz)/urdf/include/andino_materials.xacro"/> -->
 </robot>
